File: TPS63001Supply.sch (KiCad schematic (older format))
At the start: 8 parts, among them J1 Conn_01x05, U1 TPS630001

Commit message: JCLPCB
Parts:
- C1, C3, C4: LCSC (none) -> C15850
- C2: LCSC (none) -> C49678
- L1: LCSC (none) -> C341775
- R1: LCSC (none) -> C17408
- U1: value TPS630001 -> TPS63001; LCSC (none) -> C28060
Changed lines of the file:
@@
 P 5650 3450
 F 0 "U1" H 5900 3000 50  0000 C CNN
-F 1 "TPS630001" H 5650 3800 50  0000 C CNN
+F 1 "TPS63001" H 5650 3800 50  0000 C CNN
 F 2 "KevinLibrary:TPS63000" H 5650 3450 50  0001 C CNN
 F 3 "DOCUMENTATION" H 5650 3450 50  0001 C CNN
+F 4 "C28060" H 5650 3450 50  0001 C CNN "LCSC"
 	1    5650 3450
 	1    0    0    -1
@@
 Wire Wire Line
 	5650 4150 5650 4300
-$Comp
-L Device:L L1
-U 1 1 5AF900E5
-P 4500 3350
-F 0 "L1" V 4450 3350 50  0000 C CNN
-F 1 "2.2uH" V 4575 3350 50  0000 C CNN
-F 2 "Inductor_SMD:L_1210_3225Metric_Pad1.42x2.65mm_HandSolder" H 4500 3350 50  0001 C CNN
-F 3 "" H 4500 3350 50  0001 C CNN
-	1    4500 3350
-	0    -1   -1   0
-$EndComp
 Wire Wire Line
 	4850 3350 4650 3350
@@
 F 2 "Resistor_SMD:R_0805_2012Metric_Pad1.15x1.40mm_HandSolder" V 4580 4050 50  0001 C CNN
 F 3 "" H 4650 4050 50  0001 C CNN
+F 4 "C17408" V 4650 4050 50  0001 C CNN "LCSC"
 	1    4650 4050
 	1    0    0    -1
@@
 F 2 "Capacitor_SMD:C_0805_2012Metric_Pad1.15x1.40mm_HandSolder" H 4688 4500 50  0001 C CNN
 F 3 "" H 4650 4650 50  0001 C CNN
+F 4 "C49678" H 4650 4650 50  0001 C CNN "LCSC"
 	1    4650 4650
 	1    0    0    -1
@@
 F 2 "Capacitor_SMD:C_0805_2012Metric_Pad1.15x1.40mm_HandSolder" H 4088 3800 50  0001 C CNN
 F 3 "" H 4050 3950 50  0001 C CNN
+F 4 "C15850" H 4050 3950 50  0001 C CNN "LCSC"
 	1    4050 3950
 	1    0    0    -1
@@
 F 2 "Capacitor_SMD:C_0805_2012Metric_Pad1.15x1.40mm_HandSolder" H 7638 2850 50  0001 C CNN
 F 3 "" H 7600 3000 50  0001 C CNN
+F 4 "C15850" H 7600 3000 50  0001 C CNN "LCSC"
 	1    7600 3000
 	1    0    0    -1
@@
 F 2 "Capacitor_SMD:C_0805_2012Metric_Pad1.15x1.40mm_HandSolder" H 7338 2850 50  0001 C CNN
 F 3 "" H 7300 3000 50  0001 C CNN
+F 4 "C15850" H 7300 3000 50  0001 C CNN "LCSC"
 	1    7300 3000
 	1    0    0    -1
@@
 Wire Wire Line
 	7300 2750 7600 2750
+$Comp
+L Device:L L1
+U 1 1 5AF900E5
+P 4500 3350
+F 0 "L1" V 4450 3350 50  0000 C CNN
+F 1 "2.2uH" V 4575 3350 50  0000 C CNN
+F 2 "Inductor_SMD:L_1210_3225Metric_Pad1.42x2.65mm_HandSolder" H 4500 3350 50  0001 C CNN
+F 3 "" H 4500 3350 50  0001 C CNN
+F 4 "C341775" V 4500 3350 50  0001 C CNN "LCSC"
+	1    4500 3350
+	0    -1   -1   0
+$EndComp
 $EndSCHEMATC
