File: TPS63001Supply.kicad_pcb (KiCad board)
At the start: 2 copper layers, 20 x 17 mm, 9 parts, among them J1 Conn_01x05, U1 TPS630001

Commit message: Add Labels
Other:
- board text added: "EN"
- board text added: "GND"
- board text added: "PS"
- board text added: "VIN"
- board text added: "VOUT"
Changed lines of the file:
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@@
   (general
     (thickness 1.6)
-    (drawings 6)
+    (drawings 11)
     (tracks 61)
     (zones 0)
@@
     (tags "capacitor handsolder")
     (attr smd)
-    (fp_text reference C3 (at -2.6 0.1 180) (layer F.SilkS)
-      (effects (font (size 1 1) (thickness 0.15)))
+    (fp_text reference C3 (at 0 1.3 180) (layer F.SilkS)
+      (effects (font (size 0.5 0.5) (thickness 0.1)))
     )
     (fp_text value 10u (at 0 1.65 90) (layer F.Fab)
@@
     (descr "Through hole straight pin header, 1x05, 2.54mm pitch, single row")
     (tags "Through hole pin header THT 1x05 2.54mm single row")
-    (fp_text reference J1 (at 2.5 -0.3) (layer F.SilkS)
+    (fp_text reference J1 (at 0.1 -2) (layer F.SilkS)
       (effects (font (size 1 1) (thickness 0.15)))
     )
@@
     )
   )
+  (gr_text GND (at 157.2 110.1) (layer F.SilkS)
+    (effects (font (size 1 1) (thickness 0.15)))
+  )
+  (gr_text EN (at 157.6 107.6) (layer F.SilkS)
+    (effects (font (size 1 1) (thickness 0.15)))
+  )
+  (gr_text PS (at 157.6 104.9) (layer F.SilkS)
+    (effects (font (size 1 1) (thickness 0.15)))
+  )
+  (gr_text VIN (at 157.3 102.4) (layer F.SilkS)
+    (effects (font (size 1 1) (thickness 0.15)))
+  )
+  (gr_text VOUT (at 156.7 99.9) (layer F.SilkS)
+    (effects (font (size 1 1) (thickness 0.15)))
+  )
   (gr_text "TPS63001 Buck/Boost" (at 150.8 106.4) (layer B.SilkS)
     (effects (font (size 1 1) (thickness 0.25)) (justify mirror))
@@
   (segment (start 145.405 103.8552) (end 145.7566 103.5036) (width 0.3048) (layer F.Cu) (net 1))
   (segment (start 145.7566 103.5036) (end 147.495099 103.5036) (width 0.3048) (layer F.Cu) (net 1))
-  (segment (start 148.5011 105.3211) (end 149.0011 105.8211) (width 0.254) (layer F.Cu) (net 2))
-  (segment (start 149.0011 105.8211) (end 149.0011 106.5036) (width 0.254) (layer F.Cu) (net 2))
-  (segment (start 148.5011 105.0036) (end 148.5011 105.3211) (width 0.1524) (layer F.Cu) (net 2))
-  (segment (start 148.5011 103.5036) (end 148.5011 105.0036) (width 0.254) (layer F.Cu) (net 2))
   (segment (start 145.468 110.1344) (end 145.368 110.1344) (width 0.3048) (layer F.Cu) (net 1))
-  (segment (start 148.5011 107.056) (end 148.5011 107.8103) (width 0.254) (layer F.Cu) (net 3))
-  (segment (start 148.5011 106.5036) (end 148.5011 107.056) (width 0.2) (layer F.Cu) (net 3))
   (segment (start 145.1086 110.2) (end 145.043 110.1344) (width 0.3048) (layer F.Cu) (net 1))
   (segment (start 144.72 102.38) (end 144.6 102.5) (width 0.3048) (layer B.Cu) (net 1))
@@
   (segment (start 143.6198 104.0802) (end 144.6276 104.0802) (width 0.3048) (layer F.Cu) (net 1))
   (segment (start 143.2 104.5) (end 143.6198 104.0802) (width 0.3048) (layer F.Cu) (net 1))
+  (segment (start 148.5011 105.3211) (end 149.0011 105.8211) (width 0.254) (layer F.Cu) (net 2))
+  (segment (start 149.0011 105.8211) (end 149.0011 106.5036) (width 0.254) (layer F.Cu) (net 2))
+  (segment (start 148.5011 105.0036) (end 148.5011 105.3211) (width 0.1524) (layer F.Cu) (net 2))
+  (segment (start 148.5011 103.5036) (end 148.5011 105.0036) (width 0.254) (layer F.Cu) (net 2))
+  (segment (start 148.5011 107.056) (end 148.5011 107.8103) (width 0.254) (layer F.Cu) (net 3))
+  (segment (start 148.5011 106.5036) (end 148.5011 107.056) (width 0.2) (layer F.Cu) (net 3))
   (segment (start 148.5011 107.8103) (end 148.5011 109.6011) (width 0.3048) (layer F.Cu) (net 3))
   (segment (start 148.5011 109.6011) (end 149 110.1) (width 0.3048) (layer F.Cu) (net 3))
